File: pcb/keyboard.kicad_pcb (KiCad board)
At the start: 2 copper layers, 219 x 100.2 mm, 50 parts, among them J1 TRRS, SW11 1, SW12 2, SW13 3, SW14 4, SW15 5, SW16 6, SW17 7, SW18 8, SW19 9, SW21 11, SW22 12, SW23 13, SW24 14, SW25 15, SW26 16, SW27 17, SW28 18, SW29 19, SW31 21, SW32 22, SW33 23, SW34 24, SW35 25, SW36 26, SW37 27, SW38 28, SW39 29, SW41 31, SW42 32, SW43 33, SW45 35, SW46 36, SW47 37, SW48 38, SW49 39, U1 EliteC

Commit message: add lots of traces and remove solder mask from jumpers
Connections:
- U1 pad 10: ROW4 -> COL8
- U1 pad 11: LED1 -> COL9
- U1 pad 12: COL9 -> LED1
- U1 pad 13: COL8 -> COL4
- U1 pad 14: COL7 -> COL3
- U1 pad 15: COL6 -> COL2
- U1 pad 16: COL5 -> COL1
- U1 pad 17: COL4 -> ROW4
- U1 pad 18: COL3 -> ROW3
- U1 pad 19: COL2 -> ROW2
- U1 pad 20: COL1 -> ROW1
- U1 pad 7: ROW1 -> COL5
- U1 pad 8: ROW2 -> COL6
- U1 pad 9: ROW3 -> COL7
Routing:
- net (no net): track 0.00 -> 385.5 mm
- net COL6: track 0.00 -> 175.1 mm
- net ROW3: track 0.00 -> 174.9 mm
- net ROW2: track 0.00 -> 155.9 mm
- net COL5: track 0.00 -> 141.1 mm, vias 0 -> 2
- net ROW1: track 0.00 -> 141.0 mm
- net COL4: track 0.00 -> 118.9 mm, vias 0 -> 3
- net COL3: track 0.00 -> 110.4 mm, vias 0 -> 3
- net COL2: track 0.00 -> 82.9 mm, vias 0 -> 3
- net COL1: track 8.10 -> 56.8 mm, vias 1 -> 3
- net ROW4: track 0.00 -> 40.3 mm
- net Net-(SW21-Pad3): track 0.00 -> 35.1 mm
- net Net-(SW33-Pad3): track 0.00 -> 33.5 mm
- net Net-(SW32-Pad3): track 0.00 -> 33.5 mm
- net Net-(SW31-Pad3): track 0.00 -> 33.5 mm
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
Commit message: fix switch references
Parts:
- JP1, JP2: value JumperSplit -> Jumper
- SW11: value 1 -> 11
- SW12: value 2 -> 12
- SW13: value 3 -> 13
- SW14: value 4 -> 14
- SW15: value 5 -> 15
- SW16: value 6 -> 16
- SW17: value 7 -> 17
- SW18: value 8 -> 18
- SW19: value 9 -> 19
- SW21: value 11 -> 21
- SW22: value 12 -> 22
- SW23: value 13 -> 23
- SW24: value 14 -> 24
- SW25: value 15 -> 25
- SW26: value 16 -> 26
- SW27: value 17 -> 27
- SW28: value 18 -> 28
- SW29: value 19 -> 29
- SW31: value 21 -> 31
- SW32: value 22 -> 32
- SW33: value 23 -> 33
- SW34: value 24 -> 34
- SW35: value 25 -> 35
- SW36: value 26 -> 36
- SW37: value 27 -> 37
- SW38: value 28 -> 38
- SW39: value 29 -> 39
- SW41: value 31 -> 41
- SW42: value 32 -> 42
- SW43: value 33 -> 43
- SW45: value 35 -> 45
- SW46: value 36 -> 46
- SW47: value 37 -> 47
- SW48: value 38 -> 48
- SW49: value 39 -> 49
