File: left_plate/plate.kicad_sch (KiCad schematic)
At the start: 23 parts

Commit message: update plates with asymmetrical pinky stagger
Parts:
- SW16, SW26, SW35, SW36, SW45, SW46: footprint Plate:Switch -> Plate:SwitchUp
Changed lines of the file:
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@@
       (effects (font (size 1.27 1.27)))
     )
-    (property "Footprint" "Plate:Switch" (at 92.71 82.55 0)
+    (property "Footprint" "Plate:SwitchUp" (at 92.71 82.55 0)
       (effects (font (size 1.27 1.27)) hide)
     )
@@
       (effects (font (size 1.27 1.27)))
     )
-    (property "Footprint" "Plate:Switch" (at 100.33 90.17 0)
+    (property "Footprint" "Plate:SwitchUp" (at 100.33 90.17 0)
       (effects (font (size 1.27 1.27)) hide)
     )
@@
       (effects (font (size 1.27 1.27)))
     )
-    (property "Footprint" "Plate:Switch" (at 100.33 67.31 0)
+    (property "Footprint" "Plate:SwitchUp" (at 100.33 67.31 0)
       (effects (font (size 1.27 1.27)) hide)
     )
@@
       (effects (font (size 1.27 1.27)))
     )
-    (property "Footprint" "Plate:Switch" (at 100.33 82.55 0)
+    (property "Footprint" "Plate:SwitchUp" (at 100.33 82.55 0)
       (effects (font (size 1.27 1.27)) hide)
     )
@@
       (effects (font (size 1.27 1.27)))
     )
-    (property "Footprint" "Plate:Switch" (at 100.33 74.93 0)
+    (property "Footprint" "Plate:SwitchUp" (at 100.33 74.93 0)
       (effects (font (size 1.27 1.27)) hide)
     )
@@
       (effects (font (size 1.27 1.27)))
     )
-    (property "Footprint" "Plate:Switch" (at 92.71 90.17 0)
-      (effects (font (size 1.27 1.27)) hide)
-    )
+    (property "Footprint" "Plate:SwitchUp" (at 92.71 90.17 0)
+      (effects (font (size 1.27 1.27)) hide)
+    )
