File: right_plate/plate.kicad_sch (KiCad schematic)
At the start: 36 parts

Commit message: add left plate; update hole footprints; update STEP files
Parts:
- SW43, SW45, SW46, SW47, SW48, SW49: footprint Library:Switch -> Plate:Switch
Changed lines of the file:
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@@
       (effects (font (size 1.27 1.27)))
     )
-    (property "Footprint" "Library:Switch" (at 93.98 87.63 0)
+    (property "Footprint" "Plate:Switch" (at 93.98 87.63 0)
       (effects (font (size 1.27 1.27)) hide)
     )
@@
       (effects (font (size 1.27 1.27)))
     )
-    (property "Footprint" "Library:Switch" (at 116.84 87.63 0)
+    (property "Footprint" "Plate:Switch" (at 116.84 87.63 0)
       (effects (font (size 1.27 1.27)) hide)
     )
@@
       (effects (font (size 1.27 1.27)))
     )
-    (property "Footprint" "Library:Switch" (at 71.12 87.63 0)
+    (property "Footprint" "Plate:Switch" (at 71.12 87.63 0)
       (effects (font (size 1.27 1.27)) hide)
     )
@@
       (effects (font (size 1.27 1.27)))
     )
-    (property "Footprint" "Library:Switch" (at 109.22 87.63 0)
+    (property "Footprint" "Plate:Switch" (at 109.22 87.63 0)
       (effects (font (size 1.27 1.27)) hide)
     )
@@
       (effects (font (size 1.27 1.27)))
     )
-    (property "Footprint" "Library:Switch" (at 86.36 87.63 0)
+    (property "Footprint" "Plate:Switch" (at 86.36 87.63 0)
       (effects (font (size 1.27 1.27)) hide)
     )
@@
       (effects (font (size 1.27 1.27)))
     )
-    (property "Footprint" "Library:Switch" (at 101.6 87.63 0)
-      (effects (font (size 1.27 1.27)) hide)
-    )
+    (property "Footprint" "Plate:Switch" (at 101.6 87.63 0)
+      (effects (font (size 1.27 1.27)) hide)
+    )

Commit message: update plates with asymmetrical pinky stagger
Parts:
- SW16, SW26, SW35, SW36, SW45, SW46: footprint Plate:Switch -> Plate:SwitchDown
Changed lines of the file:
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@@
       (effects (font (size 1.27 1.27)))
     )
-    (property "Footprint" "Plate:Switch" (at 86.36 80.01 0)
+    (property "Footprint" "Plate:SwitchDown" (at 86.36 80.01 0)
       (effects (font (size 1.27 1.27)) hide)
     )
@@
       (effects (font (size 1.27 1.27)))
     )
-    (property "Footprint" "Plate:Switch" (at 93.98 80.01 0)
+    (property "Footprint" "Plate:SwitchDown" (at 93.98 80.01 0)
       (effects (font (size 1.27 1.27)) hide)
     )
@@
       (effects (font (size 1.27 1.27)))
     )
-    (property "Footprint" "Plate:Switch" (at 93.98 72.39 0)
+    (property "Footprint" "Plate:SwitchDown" (at 93.98 72.39 0)
       (effects (font (size 1.27 1.27)) hide)
     )
@@
       (effects (font (size 1.27 1.27)))
     )
-    (property "Footprint" "Plate:Switch" (at 93.98 64.77 0)
+    (property "Footprint" "Plate:SwitchDown" (at 93.98 64.77 0)
       (effects (font (size 1.27 1.27)) hide)
     )
@@
       (effects (font (size 1.27 1.27)))
     )
-    (property "Footprint" "Plate:Switch" (at 93.98 87.63 0)
+    (property "Footprint" "Plate:SwitchDown" (at 93.98 87.63 0)
       (effects (font (size 1.27 1.27)) hide)
     )
@@
       (effects (font (size 1.27 1.27)))
     )
-    (property "Footprint" "Plate:Switch" (at 86.36 87.63 0)
-      (effects (font (size 1.27 1.27)) hide)
-    )
+    (property "Footprint" "Plate:SwitchDown" (at 86.36 87.63 0)
+      (effects (font (size 1.27 1.27)) hide)
+    )
